File: KiCad Project/z88-internal-memory.kicad_pcb (KiCad board)
At the start: 2 copper layers, 50.8 x 44.4 mm, 12 parts, among them J1 Conn_01x02, U1 29F400, U2 IS61C5128

Commit message: progressive update
Parts:
- removed J1: Conn_01x02, Connector_PinHeader_2.54mm:PinHeader_1x02_P2.54mm_Horizontal
- C1, C2: footprint Capacitor_SMD:C_2220_5750Metric_Pad1.97x5.40mm_HandSolder -> Capacitor_SMD:C_1206_3216Metric_Pad1.33x1.80mm_HandSolder
- moved TP1 10.2 mm to (116.8, 76.2)
- moved U2 3.16 mm to (127.0, 79.3)
Connections:
- net /~{CE} renamed /~{IPCE}
- net /~{CS1} renamed /~{IRCE}
Routing:
- net VCC: track 85.4 -> 44.5 mm
- net /D1: track 51.1 -> 37.0 mm
- net /D0: track 49.0 -> 36.2 mm
- net /A0: track 56.5 -> 44.9 mm
- net /A1: track 44.5 -> 34.2 mm
- net /A2: track 34.2 -> 25.2 mm
- net /A3: track 32.9 -> 25.2 mm
- net /A4: track 31.7 -> 25.3 mm
- net /D2: track 53.2 -> 46.7 mm
- net /A5: track 30.5 -> 25.3 mm
- net /A16: track 53.9 -> 48.8 mm
- net /A12: track 39.3 -> 34.3 mm
- net /A14: track 55.5 -> 50.5 mm
- net /A6: track 30.3 -> 25.6 mm
- net /A7: track 29.5 -> 25.1 mm
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