File: KiCad Project/z88-internal-memory.kicad_sch (KiCad schematic)
At the start: 12 parts, among them J1 Conn_01x02, U1 29F400, U2 IS61C5128

Commit message: progressive update
Parts:
- added P2: ROM, Package_DIP:DIP-32_W15.24mm, symbol Z88 RAM ROM Internal:ROM_Dual_SIP16
- C1, C2: footprint Capacitor_SMD:C_2220_5750Metric_Pad1.97x5.40mm_HandSolder -> Capacitor_SMD:C_1206_3216Metric_Pad1.33x1.80mm_HandSolder
- P1: footprint Connector_SIP_Header:SIPHeader_1x16_Vertical_P1 -> Package_DIP:DIP-32_W15.24mm; symbol Z88 RAM ROM Internal:ROM Pins DIP32 -> Z88 RAM ROM Internal:ROM_Dual_SIP16
Connections:
- net ~{CE} renamed ~{IPCE}
- net ~{CS1} renamed ~{IRCE}
Other:
- moved on the sheet: C1
